File: hagiwo_osc.kicad_pcb (KiCad board)
At the start: 4 copper layers, 87.4 x 110 mm, 69 parts, among them J1 VOCT_IN, J10 OUTPUT_PIN, J11 BUTTON_PIN, J2 GAIN_IN, J3 P2_IN, J4 P1_IN, J5 MODECV_IN, J6 Eurorack Power, J7 OUT_A, J8 WIRES_TO_FRONT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

Commit message: Add voltage divider on GAIN_CV since we really need this to prevent clipping.
Parts:
- added R26: 50K, Resistor_THT:R_Axial_DIN0204_L3.6mm_D1.6mm_P2.54mm_Vertical, F.Cu at (82.3, 83.6)
- added R27: 50K, Resistor_THT:R_Axial_DIN0204_L3.6mm_D1.6mm_P2.54mm_Vertical, F.Cu at (77.2, 85.9)
- moved R2 7.44 mm to (79.8, 75.9), turned to 270 degrees
Connections:
- R2 pad 2: GAIN_IN -> Net-(R2-Pad2)
Routing:
- net Net-(R2-Pad2): track 0.00 -> 8.08 mm
